Commit message: Tiny fix in test.xacro
The line     <axis xyz="0 1 0" rpy="0 0 0"/> was missing in:

  <xacro:include filename="$(find gazebo_ros_motors)/xacro/dc_motor.xacro"/>

This would generate an "Not enough blocks" error when launching the test

File: xacro/test.xacro (robot description, xacro)
@@ -68,4 +68,5 @@
     <xacro:property name="params_yaml" value="$(find gazebo_ros_motors)/params/dc_motor.yaml"/>
     <origin xyz="0 0 0.2" rpy="0 0 0"/>
+    <axis xyz="0 1 0" rpy="0 0 0"/> <!-- Without this an Not Enough Blocks error happens -->
   </xacro:dc_motor>
 </robot>
